File: stm32f4_uno.kicad_pcb (KiCad board)
At the start: 2 copper layers, 68.6 x 53.3 mm, 66 parts, among them J1 Barrel_Jack, J101 Digital/PWM, J102 Power, J103 Analog, J104 Digital/PWM, J105 Conn_ST_STDC14, J106 Ethernet, J107 STM32 GPIO, J108 STM32 GPIO, J109 STM32 GPIO, J110 STM32 GPIO, J111 STM32 GPIO, J2 SHOU HAN TYPE-C 16PIN 2MD(073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, U101 STM32F407VGTx, U201 AMS1117-5.0, U301 AMS1117-3.3, U501 SST26VF016BEUI-104I/SN, Y101 25MHz, Y102 32.768kHz

Commit message: Set DNP on devices not to populate
Parts:
- U101: value STM32F407VGTx -> STM32F407VGT6
Changed lines of the file:
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@@
     (descr "Through hole straight socket strip, 1x08, 2.54mm pitch, single row (from Kicad 4.0.7), script generated")
     (tags "Through hole socket strip THT 1x08 2.54mm single row")
+    (property "Description" "")
+    (property "JLCPCB Part #" "")
+    (property "Manufacturer" "")
+    (property "Partnumber" "")
     (property "Sheetfile" "stm32f4_uno.kicad_sch")
     (property "Sheetname" "")
+    (property "dnp" "")
+    (property "isBasicPart" "")
     (property "ki_description" "Generic connector, single row, 01x08, script generated (kicad-library-utils/schlib/autogen/connector/)")
     (property "ki_keywords" "connector")
@@
     (descr "Through hole straight socket strip, 1x06, 2.54mm pitch, single row (from Kicad 4.0.7), script generated")
     (tags "Through hole socket strip THT 1x06 2.54mm single row")
+    (property "Description" "")
+    (property "JLCPCB Part #" "")
+    (property "Manufacturer" "")
+    (property "Partnumber" "")
     (property "Sheetfile" "stm32f4_uno.kicad_sch")
     (property "Sheetname" "")
+    (property "dnp" "")
+    (property "isBasicPart" "")
     (property "ki_description" "Generic connector, single row, 01x06, script generated (kicad-library-utils/schlib/autogen/connector/)")
     (property "ki_keywords" "connector")
@@
     (descr "Through hole straight socket strip, 1x10, 2.54mm pitch, single row (from Kicad 4.0.7), script generated")
     (tags "Through hole socket strip THT 1x10 2.54mm single row")
+    (property "Description" "")
+    (property "JLCPCB Part #" "")
+    (property "Manufacturer" "")
+    (property "Partnumber" "")
     (property "Sheetfile" "stm32f4_uno.kicad_sch")
     (property "Sheetname" "")
+    (property "dnp" "")
+    (property "isBasicPart" "")
     (property "ki_description" "Generic connector, single row, 01x10, script generated (kicad-library-utils/schlib/autogen/connector/)")
     (property "ki_keywords" "connector")
@@
     (descr "Through hole straight socket strip, 1x08, 2.54mm pitch, single row (from Kicad 4.0.7), script generated")
     (tags "Through hole socket strip THT 1x08 2.54mm single row")
+    (property "Description" "")
+    (property "JLCPCB Part #" "")
+    (property "Manufacturer" "")
+    (property "Partnumber" "")
     (property "Sheetfile" "stm32f4_uno.kicad_sch")
     (property "Sheetname" "")
+    (property "dnp" "")
+    (property "isBasicPart" "")
     (property "ki_description" "Generic connector, single row, 01x08, script generated (kicad-library-utils/schlib/autogen/connector/)")
     (property "ki_keywords" "connector")
@@
     (descr "LQFP, 100 Pin (https://www.nxp.com/docs/en/package-information/SOT407-1.pdf), generated with kicad-footprint-generator ipc_gullwing_generator.py")
     (tags "LQFP QFP")
+    (property "Description" "1MB 1.8V~3.6V ARM Cortex-M4 192KB 168MHz FLASH 82 LQFP-100(14x14)  Microcontroller Units (MCUs/MPUs/SOCs) ROHS")
+    (property "JLCPCB Part #" "C12345")
+    (property "Manufacturer" "STMicroelectronics")
+    (property "Partnumber" "STM32F407VGT6")
     (property "Sheetfile" "stm32f4_uno.kicad_sch")
     (property "Sheetname" "")
+    (property "isBasicPart" "NO")
     (property "ki_description" "STMicroelectronics Arm Cortex-M4 MCU, 1024KB flash, 192KB RAM, 168 MHz, 1.8-3.6V, 82 GPIO, LQFP100")
     (property "ki_keywords" "Arm Cortex-M4 STM32F4 STM32F407/417")
@@
         (effects (font (size 0.8 0.8) (thickness 0.13)))
     )
-    (fp_text value "STM32F407VGTx" (at 0 9.42 135) (layer "F.Fab") hide
+    (fp_text value "STM32F407VGT6" (at 0 9.42 135) (layer "F.Fab") hide
         (effects (font (size 0.8 0.8) (thickness 0.13)))
     )
@@
     (property "Sheetfile" "flash.kicad_sch")
     (property "Sheetname" "Flash (SPI)")
+    (property "dnp" "")
     (property "isBasicPart" "NO")
     (property "ki_description" "NOR-Flash 16Mbit SPI/SQI Flash w/EUI, 85C, 2.3V-3.6V")
@@
     (descr "Through hole straight socket strip, 1x08, 2.54mm pitch, single row (from Kicad 4.0.7), script generated")
     (tags "Through hole socket strip THT 1x08 2.54mm single row")
+    (property "Description" "")
+    (property "JLCPCB Part #" "")
+    (property "Manufacturer" "")
+    (property "Partnumber" "")
     (property "Sheetfile" "stm32f4_uno.kicad_sch")
     (property "Sheetname" "")
+    (property "dnp" "")
+    (property "isBasicPart" "")
     (property "ki_description" "Generic connector, single row, 01x08, script generated (kicad-library-utils/schlib/autogen/connector/)")
     (property "ki_keywords" "connector")
@@
     (descr "Through hole straight socket strip, 1x08, 2.54mm pitch, single row (from Kicad 4.0.7), script generated")
     (tags "Through hole socket strip THT 1x08 2.54mm single row")
+    (property "Description" "")
+    (property "JLCPCB Part #" "")
+    (property "Manufacturer" "")
+    (property "Partnumber" "")
     (property "Sheetfile" "stm32f4_uno.kicad_sch")
     (property "Sheetname" "")
+    (property "dnp" "")
+    (property "isBasicPart" "")
     (property "ki_description" "Generic connector, single row, 01x08, script generated (kicad-library-utils/schlib/autogen/connector/)")
     (property "ki_keywords" "connector")
@@
     (descr "Through hole straight socket strip, 1x06, 2.54mm pitch, single row (from Kicad 4.0.7), script generated")
     (tags "Through hole socket strip THT 1x06 2.54mm single row")
+    (property "Description" "")
+    (property "JLCPCB Part #" "")
+    (property "Manufacturer" "")
+    (property "Partnumber" "")
     (property "Sheetfile" "stm32f4_uno.kicad_sch")
     (property "Sheetname" "")
+    (property "dnp" "")
+    (property "isBasicPart" "")
     (property "ki_description" "Generic connector, single row, 01x06, script generated (kicad-library-utils/schlib/autogen/connector/)")
     (property "ki_keywords" "connector")
@@
     (property "Sheetfile" "stm32f4_uno.kicad_sch")
     (property "Sheetname" "")
+    (property "dnp" "")
     (property "isBasicPart" "")
     (property "ki_description" "Generic connector, single row, 01x10, script generated (kicad-library-utils/schlib/autogen/connector/)")
@@
     (descr "Through hole straight socket strip, 1x08, 2.54mm pitch, single row (from Kicad 4.0.7), script generated")
     (tags "Through hole socket strip THT 1x08 2.54mm single row")
+    (property "Description" "")
+    (property "JLCPCB Part #" "")
+    (property "Manufacturer" "")
+    (property "Partnumber" "")
     (property "Sheetfile" "stm32f4_uno.kicad_sch")
     (property "Sheetname" "")
+    (property "dnp" "")
+    (property "isBasicPart" "")
     (property "ki_description" "Generic connector, single row, 01x08, script generated (kicad-library-utils/schlib/autogen/connector/)")
     (property "ki_keywords" "connector")
@@
     (descr "Through hole straight socket strip, 1x08, 2.54mm pitch, single row (from Kicad 4.0.7), script generated")
     (tags "Through hole socket strip THT 1x08 2.54mm single row")
+    (property "Description" "")
+    (property "JLCPCB Part #" "")
+    (property "Manufacturer" "")
+    (property "Partnumber" "")
     (property "Sheetfile" "stm32f4_uno.kicad_sch")
     (property "Sheetname" "")
+    (property "dnp" "")
+    (property "isBasicPart" "")
     (property "ki_description" "Generic connector, single row, 01x08, script generated (kicad-library-utils/schlib/autogen/connector/)")
     (property "ki_keywords" "connector")

Commit message: #1 Use new central library KiCad-Lib
Parts:
- J105: footprint Project_Library:Samtec_FTSH-107-XX-YYY-DV-K -> #Connector_Debug:Amphenol ICC 20021511-00014T4LF
- J2: footprint Project_Library:SHOU HAN TYPE-C 16PIN 2MD(073) (C2765186) -> #Connector:SHOU HAN TYPE-C 16PIN 2MD(073)
- moved J105 7.84 mm to (165.6, 79.6)
Routing:
- net /~{RESET}: track 65.6 -> 54.4 mm, vias 4 -> 3
- net +3V3: track 243.2 -> 248.7 mm, vias 10 -> 8
- net /USART1_TX: track 43.0 -> 48.0 mm
- net /SYS_SWO: track 29.6 -> 34.5 mm
- net /SYS_SWDIO: track 29.9 -> 34.3 mm
- net /SYS_SWCLK: track 30.0 -> 34.1 mm
- net GND: track 68.0 -> 66.8 mm, vias 20 -> 19
- net /USART1_RX: track 37.6 -> 36.5 mm, vias 2 -> 1
